Commit message: fix urdf errors

File: gazebo-arm.urdf.xacro (robot description, xacro)
@@ -1,5 +1,5 @@
 <?xml version="1.0"?>
 <robot name="arm" xmlns:xacro="http://www.ros.org/wiki/xacro">
-		<xacro:include filename="$(find robond_rl)/urdf/gazebo_arm.gazebo" />
+		<xacro:include filename="$(find robond-rl)/urdf/gazebo-arm.gazebo" />
 		<link name="base">
 			<pose>0 0 .1 0 0 0</pose>
@@ -102,10 +102,10 @@
 			<visual>
 			  <geometry>
-				<mesh filename="package://robond_rl/meshes/gripper/gripper_base.dae"/>
+				<mesh filename="package://robond-rl/meshes/gripper/gripper_base.dae"/>
 			  </geometry>
 			</visual>
 			<collision>
 			  <geometry>
-				<mesh filename="package://robond_rl/meshes/gripper/gripper_base.dae"/>
+				<mesh filename="package://robond-rl/meshes/gripper/gripper_base.dae"/>
 			  </geometry>
 			</collision>
@@ -120,10 +120,10 @@
 		  <origin xyz="0 0 0" rpy="0 0 0"/>
 		  <geometry>
-			<mesh filename="package://robond_rl/meshes/gripper/finger_right.dae"/>
+			<mesh filename="package://robond-rl/meshes/gripper/finger_right.dae"/>
 		  </geometry>
 		</visual>
 		<collision>
 		  <geometry>
-			<mesh filename="package://robond_rl/meshes/gripper/finger_right_collision.dae"/>
+			<mesh filename="package://robond-rl/meshes/gripper/finger_right_collision.dae"/>
 		  </geometry>
 		</collision>
@@ -137,10 +137,10 @@
 		<visual>
 		  <geometry>
-			<mesh filename="package://robond_rl/meshes/gripper/finger_left.dae"/>
+			<mesh filename="package://robond-rl/meshes/gripper/finger_left.dae"/>
 		  </geometry>
 		</visual>
 		<collision>
 		  <geometry>
-			<mesh filename="package://robond_rl/meshes/gripper/finger_left_collision.dae"/>
+			<mesh filename="package://robond-rl/meshes/gripper/finger_left_collision.dae"/>
 		  </geometry>
 		</collision>
@@ -167,5 +167,5 @@
 		<child link="base"/>
 		<origin xyz="0 0 0" rpy="0 0 0"/>
-		<limit upper="2" lower="-2" </>
+		<limit upper="2" lower="-2" />
 		<axis xyz="0 0 1" />
 	  </joint>
@@ -174,5 +174,5 @@
 		<child link="joint1"/>
 		<origin xyz="0 0 0" rpy="0 0 0"/>
-		<limit upper="2" lower="-2" </>
+		<limit upper="2" lower="-2" />
 		<axis xyz="0 1 0" />
 	  </joint>
@@ -181,5 +181,5 @@
 		<child link="link1"/>
 		<origin xyz="0 0 -0.05" rpy="0 0 0"/>
-		<limit upper="0" lower="0" </>
+		<limit upper="0" lower="0" />
 		<axis xyz="0 1 0" />
 	  </joint>
@@ -188,5 +188,5 @@
 		<child link="joint2"/>
 		<origin xyz="0 0 -0.05" rpy="0 0 0"/>
-		<limit upper="2" lower="-2" </>
+		<limit upper="2" lower="-2" />
 		<axis xyz="0 1 0" />
 	  </joint>
@@ -195,5 +195,5 @@
 		<child link="link2"/>
 		<origin xyz="0 0 -0.05" rpy="0 0 0"/>
-		<limit upper="0" lower="0" </>
+		<limit upper="0" lower="0" />
 		<axis xyz="0 1 0" />
 	  </joint>
@@ -223,5 +223,5 @@
 		<parent link="gripperbase"/>
 		<child link="gripper_middle"/>
-		<origin xyz="0 0 0 rpy="0 0 0"/>
+		<origin xyz="0 0 0" rpy="0 0 0"/>
 		<axis xyz="0 1 0" />
 	  </joint>

Commit message: update joint limit effort and velocity values

File: gazebo-arm.urdf.xacro (robot description, xacro)
@@ -174,5 +174,5 @@
 		<child link="joint1"/>
 		<origin xyz="0 0 0" rpy="0 0 0"/>
-		<limit upper="2" lower="-2" />
+		<limit effort="30" velocity="0.017453293*120" upper="2" lower="-2" />
 		<axis xyz="0 1 0" />
 	  </joint>
@@ -181,5 +181,5 @@
 		<child link="link1"/>
 		<origin xyz="0 0 -0.05" rpy="0 0 0"/>
-		<limit upper="0" lower="0" />
+		<limit effort="30" velocity="0.017453293*120" upper="0" lower="0" />
 		<axis xyz="0 1 0" />
 	  </joint>
@@ -188,5 +188,5 @@
 		<child link="joint2"/>
 		<origin xyz="0 0 -0.05" rpy="0 0 0"/>
-		<limit upper="2" lower="-2" />
+		<limit effort="30" velocity="0.017453293*120" upper="2" lower="-2" />
 		<axis xyz="0 1 0" />
 	  </joint>
@@ -195,5 +195,5 @@
 		<child link="link2"/>
 		<origin xyz="0 0 -0.05" rpy="0 0 0"/>
-		<limit upper="0" lower="0" />
+		<limit effort="30" velocity="0.017453293*120" upper="0" lower="0" />
 		<axis xyz="0 1 0" />
 	  </joint>
